Commit message: Exported walking policies with a deploy contract; the D1 on its measured mount and base
Walking policies (rescue_sim):
- policies/go2_policies_2026-09-18: the flat and rough Go2 policies exported from the
  Go2_RL_workflow project, each with policy.pt/.onnx and params/{deploy,env,agent}.yaml, and
  the bundle's own deploy_contract.py reader.
- rescue_sim/exported_policy.py builds an exported policy's observation from its contract,
  instead of the sim's 235-wide layout. It uses the recorded term order, scales, clips and
  command envelope, and, for the rough policy, a camera-masked height scan rebuilt from the
  bundle's description. `--policy DIR` selects it; env_cfg.py, sim.py, the README and
  agent_cfg.py carry the wiring. Tests are in tests/test_exported_policy.py.

The D1, measured on the real arm (2026-09-30, same change as D1Training's):
- arm_weld.D1_MOUNT_POS = (-0.019, 0, 0.0855). The arm bolts through the rails' own
  screw positions (its holes 13 cm apart, the rail screws 131.0 mm apart), centred between
  them on the rail tops. It replaces (0, 0, 0.08). omniverse_sim.py (weld, teleport offset
  and reach clamp), training/go2_rescue/welded_robot.py and rescue_sim/sim.py use it.
- d1_arm: the real base is 126 mm across and 76 mm to the rotating plate, where Unitree's
  model is 105 mm and 53.3 mm. measured_base.py writes base_link_measured.STL, and d1.urdf
  uses it with Joint1 at 76.0 mm. The files are byte-identical with D1Training's.
- Policies trained before this carried the arm 19 mm further forward and 28.2 mm lower at the
  shoulder.

Co-Authored-By: Claude Opus 5.5 <noreply@anthropic.com>

File: Isaac/go2_omniverse/d1_arm/d1.urdf (robot description, URDF)
Before this commit: robot d1_description, 9 links, 8 joints
Links:
- link base_link: geometry collision mesh filename=meshes/base_link_measured.STL; visual mesh filename=meshes/base_link_measured.STL
Joints:
- joint Joint1: origin xyz=0 0 0.0533 rpy=0 0 -3.1416 -> xyz=0 0 0.076 rpy=0 0 -3.1416

Commit message: The D1 from D1Training's latest model, and the Go2 EDU's dock drawn under it
The arm (d1_arm/, byte-identical with D1Training's working tree at 054983a, 2026-10-09):
- Unitree's D1-550 CAD joint lengths above Joint1 (D1Training F-138): the shoulder 54.8 mm above Joint1, the upper
  arm 270.0 mm, the forearm 204.67 mm to Joint5, the fingertips 206.38 mm past it.
- The measured base's mounting holes 58 mm across the rail, as Unitree's (measured_base.py keeps the flange's tabs at
  Unitree's width).
- Joint2 and Joint3 limited at 3.33 N*m, as Unitree's D1-550 URDF has them (F-137; not measured), in d1.urdf and
  rescue_sim/d1_model.py. The parity fixture is regenerated from D1Training (make_fixtures.py now records a dirty
  tree as such).

The dock: dock.py and dock_meshes/ (D1Training's dock.py and Unitree-CAD meshes, with their NOTICE; no licence is
stated for the CAD). arm_weld.py draws the expansion dock and its rails on the trunk, visual only, as D1Training's
weld.py does; `dock_visual=False` leaves them out (training, where 20k triangles a robot is 82M across 4096).

The wrist RealSense and its mount were already D1Training's and are unchanged.

Co-Authored-By: Claude Opus 5.5 (1M context) <noreply@anthropic.com>

File: Isaac/go2_omniverse/d1_arm/d1.urdf (robot description, URDF)
Before this commit: robot d1_description, 9 links, 8 joints
Joints:
- joint Joint2: limit lower=-1.57 upper=1.57 effort=3.3 velocity=1.05 -> lower=-1.57 upper=1.57 effort=3.33 velocity=1.05; origin xyz=0 0.028 0.0563 rpy=1.5708 0 -3.1416 -> xyz=0 0.028 0.0548 rpy=1.5708 0 -3.1416
- joint Joint3: limit lower=-1.57 upper=1.57 effort=1.7 velocity=1.05 -> lower=-1.57 upper=1.57 effort=3.33 velocity=1.05; origin xyz=0 0.2693 0.0009 rpy=0 0 0 -> xyz=0 0.27 0 rpy=0 0 0
- joint Joint4: origin xyz=0.0577 0.042 -0.0275 rpy=-1.5708 0 -1.5708 -> xyz=0.0577 0.041325 -0.0275 rpy=-1.5708 0 -1.5708
- joint Joint5: origin xyz=-0.0001 -0.0237 0.14018 rpy=1.5708 -1.5708 0 -> xyz=-0.0001 -0.0237 0.146973 rpy=1.5708 -1.5708 0
- joint Joint6: origin xyz=0.0825 -0.0010782 -0.023822 rpy=-1.5708 0 -1.5708 -> xyz=0.080781 -0.0010782 -0.023822 rpy=-1.5708 0 -1.5708
